Commit message: added COARSE camera transform and launch file for tf publisher

File: description/ros2_control/padman.ros2_control.xacro (robot description, xacro)
@@ -14,4 +14,8 @@
           <param name="max">1</param>
         </command_interface>
+        <command_interface name="effort">
+          <param name="min">-0.1</param>
+          <param name="max">0.1</param>
+        </command_interface>
         <state_interface name="position"/>
       </joint>
@@ -20,4 +24,8 @@
           <param name="min">-1</param>
           <param name="max">1</param>
+        </command_interface>
+        <command_interface name="effort">
+          <param name="min">-0.1</param>
+          <param name="max">0.1</param>
         </command_interface>
         <state_interface name="position"/>
@@ -28,4 +36,8 @@
           <param name="max">1</param>
         </command_interface>
+        <command_interface name="effort">
+          <param name="min">-0.1</param>
+          <param name="max">0.1</param>
+        </command_interface>
         <state_interface name="position"/>
       </joint>

File: description/urdf/padman_description.urdf.xacro (robot description, xacro)
@@ -207,5 +207,5 @@
 </transmission>
 <joint name="Rigid_10" type="fixed">
-  <origin xyz="0.012947 0.022198 0.14824" rpy="0 0 0"/>
+  <origin xyz="0.0 0.085 0.0" rpy="0 0 0"/>
   <parent link="link22"/>
   <child link="ee1"/>

Commit message: urdf

File: description/ros2_control/padman.ros2_control.xacro (robot description, xacro)
@@ -19,4 +19,5 @@
         </command_interface>
         <state_interface name="position"/>
+        <state_interface name="velocity"/>
       </joint>
       <joint name="${prefix}joint2">
@@ -30,4 +31,5 @@
         </command_interface>
         <state_interface name="position"/>
+        <state_interface name="velocity"/>
       </joint>
         <joint name="${prefix}joint3">
@@ -41,4 +43,5 @@
         </command_interface>
         <state_interface name="position"/>
+        <state_interface name="velocity"/>
       </joint>
     </ros2_control>

File: description/urdf/padman.urdf (robot description, URDF)
Before this commit: robot arm2urdf, 4 links, 3 joints
Links:
- added link ee1, mass 0.0; collision mesh filename=file:///home/manuelbaum/ws_control/install/padman_hw/share/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 scale=0.001 0.001 0.001; visual mesh filename=file:///home/manuelbaum/ws_control/install/padman_hw/share/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 scale=0.001 0.001 0.001
- added link link01gb2, mass 0.6868164549052078; collision mesh filename=file:///home/manuelbaum/ws_control/install/padman_hw/share/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 scale=0.001 0.001 0.001; visual mesh filename=file:///home/manuelbaum/ws_control/install/padman_hw/share/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 scale=0.001 0.001 0.001
- added link link11gb4106_padman_v71, mass 0.1050227832534516; collision mesh filename=file:///home/manuelbaum/ws_control/install/padman_hw/share/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 scale=0.001 0.001 0.001; visual mesh filename=file:///home/manuelbaum/ws_control/install/padman_hw/share/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 scale=0.001 0.001 0.001
- added link world
- link base_link: mass 0.6868164549052078 -> 0.6868164549052079; geometry collision mesh filename=file:///home/manuelbaum/ws_control/install/padman_hw/share/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 scale=0.001 0.001 0.001; visual mesh filename=file:///home/manuelbaum/ws_control/install/padman_hw/share/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 scale=0.001 0.001 0.001
- link link01: mass 1.5574162139522874 -> 1.557417461604787; geometry collision mesh filename=file:///home/manuelbaum/ws_control/install/padman_hw/share/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 scale=0.001 0.001 0.001; visual mesh filename=file:///home/manuelbaum/ws_control/install/padman_hw/share/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 scale=0.001 0.001 0.001
- link link11: mass 0.6848943201158626 -> 0.6848943201158819; geometry collision mesh filename=file:///home/manuelbaum/ws_control/install/padman_hw/share/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 scale=0.001 0.001 0.001; visual mesh filename=file:///home/manuelbaum/ws_control/install/padman_hw/share/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 scale=0.001 0.001 0.001
- link link22: mass 0.06355160747290721 -> 0.0635516074729072; geometry collision mesh filename=file:///home/manuelbaum/ws_control/install/padman_hw/share/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 scale=0.001 0.001 0.001; visual mesh filename=file:///home/manuelbaum/ws_control/install/padman_hw/share/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 scale=0.001 0.001 0.001
Joints:
- removed joint Revolute_7
- removed joint Revolute_8
- removed joint Revolute_9
- added joint Rigid_10: type fixed, parent link22, child ee1, origin xyz=0.0 0.085 0.0 rpy=0 0 0
- added joint base_joint: type fixed, parent world, child base_link, origin xyz=0 0 0 rpy=0 0 0
- added joint joint1: type revolute, parent base_link, child link01, origin xyz=-0.05375 0.036 0.0 rpy=0 0 0, axis 0.0 1.0 0.0, limit lower=-2.094395 upper=1.047198 effort=100 velocity=100
- added joint joint2: type revolute, parent link01gb2, child link11, origin xyz=0.0 0.0 -0.0415 rpy=0 0 0, axis 0.0 -0.0 1.0, limit lower=-2.094395 upper=1.047198 effort=100 velocity=100
- added joint joint3: type revolute, parent link11gb4106_padman_v71, child link22, origin xyz=0.0 0.0 -0.027227 rpy=0 0 0, axis -0.0 0.0 1.0, limit lower=-2.094395 upper=1.047198 effort=100 velocity=100
- added joint link01_Rigid 1: type fixed, parent link01, child link01gb2, origin xyz=0.0 0.088937 -0.002387 rpy=0 0 0
- added joint link11_Rigid 1: type fixed, parent link11, child link11gb4106_padman_v71, origin xyz=-0.027255 0.096215 -0.011 rpy=0 0 0

Commit message: now hardware with two arms works

File: description/ros2_control/padman.ros2_control.xacro (robot description, xacro)
@@ -9,5 +9,5 @@
         <param name="example_param_hw_slowdown">100</param>
       </hardware>
-      <joint name="${prefix}joint1">
+      <joint name="${prefix}joint1_l">
         <command_interface name="position">
           <param name="min">-1</param>
@@ -21,5 +21,5 @@
         <state_interface name="velocity"/>
       </joint>
-      <joint name="${prefix}joint2">
+      <joint name="${prefix}joint2_l">
         <command_interface name="position">
           <param name="min">-1</param>
@@ -33,5 +33,41 @@
         <state_interface name="velocity"/>
       </joint>
-        <joint name="${prefix}joint3">
+        <joint name="${prefix}joint3_l">
+        <command_interface name="position">
+          <param name="min">-1</param>
+          <param name="max">1</param>
+        </command_interface>
+        <command_interface name="effort">
+          <param name="min">-0.1</param>
+          <param name="max">0.1</param>
+        </command_interface>
+        <state_interface name="position"/>
+        <state_interface name="velocity"/>
+      </joint>
+      <joint name="${prefix}joint1_r">
+        <command_interface name="position">
+          <param name="min">-1</param>
+          <param name="max">1</param>
+        </command_interface>
+        <command_interface name="effort">
+          <param name="min">-0.1</param>
+          <param name="max">0.1</param>
+        </command_interface>
+        <state_interface name="position"/>
+        <state_interface name="velocity"/>
+      </joint>
+      <joint name="${prefix}joint2_r">
+        <command_interface name="position">
+          <param name="min">-1</param>
+          <param name="max">1</param>
+        </command_interface>
+        <command_interface name="effort">
+          <param name="min">-0.1</param>
+          <param name="max">0.1</param>
+        </command_interface>
+        <state_interface name="position"/>
+        <state_interface name="velocity"/>
+      </joint>
+        <joint name="${prefix}joint3_r">
         <command_interface name="position">
           <param name="min">-1</param>

File: description/urdf/padman.urdf.xacro (robot description, xacro)
@@ -4,4 +4,5 @@
   <!-- Import RRBot macro -->
   <xacro:include filename="$(find padman_hw)/urdf/padman_description.urdf.xacro" />
+  <xacro:include filename="$(find padman_hw)/urdf/padman_description_right.urdf.xacro" />
   <!-- Import Rviz colors -->
   <!--<xacro:include filename="$(find padman_hw)/padman/urdf/padman.materials.xacro" />-->
@@ -13,4 +14,7 @@
     <origin xyz="0 0 0" rpy="0 0 0" />
   </xacro:padman>
+  <xacro:padman_right parent="base_link" prefix="$(arg prefix)">
+    <origin xyz="0.255 0 0" rpy="0 0 0" />
+  </xacro:padman_right>
   <xacro:padman_ros2_control
     name="Padman" prefix="$(arg prefix)" />

File: description/urdf/padman_description.urdf.xacro (robot description, xacro)
@@ -120,5 +120,5 @@
   <child link="ee1"/>
 </joint>
-<joint name="joint2" type="revolute">
+<joint name="joint2_l" type="revolute">
   <origin xyz="0.0 0.088937 -0.043887" rpy="0 0 0"/>
   <parent link="link01"/>
@@ -137,5 +137,5 @@
   </actuator>
 </transmission>
-<joint name="joint1" type="revolute">
+<joint name="joint1_l" type="revolute">
   <origin xyz="-0.05375 0.036 0.0" rpy="0 0 0"/>
   <parent link="base_link"/>
@@ -154,5 +154,5 @@
   </actuator>
 </transmission>
-<joint name="joint3" type="revolute">
+<joint name="joint3_l" type="revolute">
   <origin xyz="0.002293 0.099974 -0.037727" rpy="0 0 0"/>
   <parent link="link11"/>
